File: hardware/hackrf-one-plus/baseband.kicad_sch (KiCad schematic)
At the start: 136 parts, among them P14 XCVR_CLKOUT, P15 INTR, P18 OEB, P37 SCL, P38 SDA, P39 SSP1_SCK, P40 SSP1_COPI, P41 SSP1_CIPO, P53 CS_XCVR, P54 CS_AD, P55 TXENABLE, P56 RXENABLE, P57 XTAL2, P58 GCK1, P59 GCK2, P60 SGPIO_CLK, P61 DA0, P62 DA7, P63 DD0, P64 DD9, P65 DA4, P66 DD5, P67 RSSI, P83 GND, P84 GND, P85 GND, P86 GND, P87 GND, P88 GND, P89 GND, P90 GND, P91 GND, P92 GND

Commit message: feat: convert layer 3 from power to ground
Parts:
- C100, C97, C98: value (none) -> 330nF; footprint (none) -> hackrf:GSG-0402
- C101, C102, C103, C107, C108, C109, C110, C84, C85, C86, C94, C95, C96, C99: value (none) -> 22pF; footprint (none) -> hackrf:GSG-0402
- C104, C111: value (none) -> 3pF; footprint (none) -> hackrf:GSG-0402
- C105: value (none) -> 10uF; footprint (none) -> hackrf:GSG-0805
- C106: value (none) -> 1uF; footprint (none) -> hackrf:GSG-0402
- C112: value (none) -> 180pF; footprint (none) -> hackrf:GSG-0402
- C113, C119, C120, C121, C122, C123, C167, C71, C73, C75, C77, C79, C81, C83, C91: value (none) -> 100nF; footprint (none) -> hackrf:GSG-0402
- C114: value (none) -> 3.3nF; footprint (none) -> hackrf:GSG-0402
- C115: value (none) -> 33pF; footprint (none) -> hackrf:GSG-0402
- C116: value (none) -> 47pF; footprint (none) -> hackrf:GSG-0402
- C124, C72, C74, C76, C78, C80, C82: value (none) -> 2.2uF; footprint (none) -> hackrf:GSG-0402
- C159, C165, C168, C68, C69, C90: value (none) -> 100pF; footprint (none) -> hackrf:GSG-0402
- C169, C170: value (none) -> 1.8pF; footprint (none) -> hackrf:GSG-0402
- C87, C88, C89, C92, C93: value (none) -> 10nF; footprint (none) -> hackrf:GSG-0402
- D3, D9: value (none) -> GSG-DIODE-TVS-BI; footprint (none) -> hackrf:GSG-0402
- FB2: value (none) -> FILTER; footprint (none) -> hackrf:GSG-0805
- L6, L8, L9: value (none) -> DNP; footprint (none) -> hackrf:GSG-0402
- L7: value (none) -> 6.2nH; footprint (none) -> hackrf:GSG-0402
- NT3: value (none) -> VAA; footprint (none) -> gsg-modules:HEADER-1x2-SHORTED
- P16: value (none) -> CLKIN; footprint (none) -> hackrf:GSG-SMA-73251-2120
- P2: value (none) -> CLKOUT; footprint (none) -> hackrf:GSG-SMA-73251-2120
- P9: value (none) -> BASEBAND; footprint (none) -> hackrf:GSG-HEADER-2x8
- Q3: value (none) -> MOSFET_P; footprint (none) -> gsg-modules:SOT23-3
- R10, R13, R8, R9: value (none) -> 1k; footprint (none) -> hackrf:GSG-0402
- R104, R105, R11, R41, R85: value (none) -> 10k; footprint (none) -> hackrf:GSG-0402
- R14, R15, R16, R17: value (none) -> 4k7; footprint (none) -> hackrf:GSG-0402
- R20, R21, R22, R23: value (none) -> 0; footprint (none) -> hackrf:GSG-0402
- R25, R26: value (none) -> 475; footprint (none) -> hackrf:GSG-0402
- R27, R28: value (none) -> 1k8; footprint (none) -> hackrf:GSG-0402
- R31, R32, R33, R94: value (none) -> 39; footprint (none) -> hackrf:GSG-0402
- T3: value (none) -> RX_BALUN; footprint (none) -> hackrf:GSG-2500BL14M100
- T4: value (none) -> TX_BALUN; footprint (none) -> hackrf:GSG-2500BL14M100
- U17: value (none) -> MAX2837; footprint (none) -> hackrf:GSG-QFN48-6
- U18: value (none) -> MAX5864; footprint (none) -> hackrf:GSG-QFN48-7
- U19: value (none) -> SI5351C; footprint (none) -> hackrf:GSG-QFN20-4
- X1: value (none) -> GSG-XTAL4PIN; footprint (none) -> hackrf:GSG-XTAL3.2x2.5mm
