File: hardware/hackrf-one-plus/frontend.kicad_sch (KiCad schematic)
At the start: 143 parts, among them J10 GND_CLIP, J4 MOUNTING_HOLE, J5 MOUNTING_HOLE, J6 MOUNTING_HOLE, J7 MOUNTING_HOLE, J8 MOUNTING_HOLE, J9 MOUNTING_HOLE, P13 GPO1, P17 GPO6, P19 GPO3, P21 REF_IN, P27 MIXER_SDATA, P31 MIXER_SCLK, P32 MIXER_ENX, P33 MIXER_RESETX, P34 MIX_BYPASS, P35 !MIX_BYPASS, P43 RX, P44 HP, P45 LP, P46 TX_MIX_BP, P47 RX_MIX_BP, P48 TX_AMP, P49 RX_AMP, P50 AMP_BYPASS, P51 !TX_AMP_PWR, P52 !RX_AMP_PWR, P6 GPO4, P7 GPO2

Commit message: feat: convert layer 3 from power to ground
Parts:
- C1, C11, C24, C29, C3, C33, C34, C35, C36, C37, C38, C39, C40, C45, C47, C5, C55, C57, C60, C63, C65, C66, C67, C7: value (none) -> 33pF; footprint (none) -> hackrf:GSG-0402
- C10, C16, C162, C163, C19, C2, C22, C30, C4, C54, C56, C6: value (none) -> 10nF; footprint (none) -> hackrf:GSG-0402
- C12, C13: value (none) -> 330pF; footprint (none) -> hackrf:GSG-0402
- C14: value (none) -> 8p2; footprint (none) -> hackrf:GSG-0402
- C15: value (none) -> 180pF; footprint (none) -> hackrf:GSG-0402
- C160, C41, C42, C52, C70: value (none) -> 100pF; footprint (none) -> hackrf:GSG-0402
- C161, C171, C53: value (none) -> 1uF; footprint (none) -> hackrf:GSG-0402
- C166, C17, C18, C20, C23, C25, C28, C31, C44, C46, C49, C50, C58, C59, C61, C62, C64, C9: value (none) -> 100nF; footprint (none) -> hackrf:GSG-0402
- C21, C32, C43, C48, C51, C8: value (none) -> 22pF; footprint (none) -> hackrf:GSG-0402
- C26, C27: value (none) -> 47pF; footprint (none) -> hackrf:GSG-0402
- D1: value (none) -> GSG-DIODE-TVS-BI; footprint (none) -> hackrf:GSG-0402
- J2: value (none) -> RF-SHIELD-FRAME; footprint (none) -> hackrf:GSG-SHIELD-BMI-S-230
- J3: value (none) -> RF-SHIELD-COVER; footprint (none) -> hackrf:GSG-NULL-MODULE
- L1, L4: value (none) -> DNP; footprint (none) -> hackrf:GSG-0402
- L12, L13, L2, L3, L5: value (none) -> 10uH; footprint (none) -> hackrf:GSG-0603
- P4: value (none) -> ANTENNA; footprint (none) -> hackrf:GSG-SMA-73251-2120
- Q1, Q2, Q4: value (none) -> MOSFET_P; footprint (none) -> gsg-modules:SOT23-3
- R1, R2: value (none) -> 470; footprint (none) -> hackrf:GSG-0402
- R24, R29, R36, R5, R6: value (none) -> 10k; footprint (none) -> hackrf:GSG-0402
- R3: value (none) -> 22k; footprint (none) -> hackrf:GSG-0402
- R4: value (none) -> 51k; footprint (none) -> hackrf:GSG-0402
- T1: value (none) -> MIX_IN_BALUN; footprint (none) -> hackrf:GSG-B0310J50100AHF
- T2: value (none) -> MIX_OUT_BALUN; footprint (none) -> hackrf:GSG-B0310J50100AHF
- U1, U10, U11, U2, U5, U6, U7: value (none) -> SKY13453; footprint (none) -> gsg-modules:SKY13350-385LF
- U12, U14, U9: value (none) -> SKY13317; footprint (none) -> hackrf:GSG-SKY13317-373LF
- U13, U25: value (none) -> MGA-81563; footprint (none) -> hackrf:GSG-SOT363
- U3: value (none) -> RX_LOWPASS_FILTER; footprint (none) -> hackrf:GSG-LP0603
- U4: value (none) -> RFFC5072; footprint (none) -> hackrf:GSG-QFN32
- U8: value (none) -> RX_HIGHPASS_FILTER; footprint (none) -> hackrf:GSG-HP-DEA
