File: hardware/hackrf-one-plus/mcu.kicad_sch (KiCad schematic)
At the start: 134 parts, among them P23 DBGEN, P24 TRST, P68 SPIFI_CS, P69 VREGMODE, P70 EN_1V8, P71 ID, P72 GP_CLKIN, P73 P1_2, P74 P1_1, P75 GP_CLKIN, P76 GP_CLKIN, P77 GP_CLKIN, P78 GP_CLKIN, P79 GP_CLKIN, P81 SPIFI_SIO2, P82 SPIFI_SIO3

Commit message: feat: convert layer 3 from power to ground
Parts:
- C118, C157, C158, C164: value (none) -> 18pF; footprint (none) -> hackrf:GSG-0402
- C125: value (none) -> 33pF; footprint (none) -> hackrf:GSG-0402
- C126, C127, C143, C145, C146: value (none) -> 10uF; footprint (none) -> hackrf:GSG-0805
- C128, C129, C130, C131, C132, C133, C134, C135, C136, C137, C138, C139, C140, C141, C142, C144, C147, C148, C149, C150, C151, C152, C153, C154: value (none) -> 100nF; footprint (none) -> hackrf:GSG-0402
- C155, R35: value (none) -> DNP; footprint (none) -> hackrf:GSG-0805
- C156: value (none) -> 47pF; footprint (none) -> hackrf:GSG-0402
- D2: value (none) -> VAALED; footprint (none) -> gsg-modules:LTST-S220
- D4: value (none) -> USBLED; footprint (none) -> gsg-modules:LTST-S220
- D5: value (none) -> RXLED; footprint (none) -> gsg-modules:LTST-S220
- D6: value (none) -> TXLED; footprint (none) -> gsg-modules:LTST-S220
- D7: value (none) -> VCCLED; footprint (none) -> gsg-modules:LTST-S220
- D8: value (none) -> 1V8LED; footprint (none) -> gsg-modules:LTST-S220
- FB1, FB3: value (none) -> FILTER; footprint (none) -> hackrf:GSG-0805
- J1: value (none) -> USB-MICRO-B; footprint (none) -> hackrf:GSG-USB-MICROB-FCI-10103592-EXT
- L10, L11: value (none) -> 4u7; footprint (none) -> hackrf:GSG-NRG4026
- NT1: value (none) -> 1V8; footprint (none) -> gsg-modules:HEADER-1x2-SHORTED
- NT2: value (none) -> VCC; footprint (none) -> gsg-modules:HEADER-1x2-SHORTED
- P20: value (none) -> GPIO; footprint (none) -> hackrf:GSG-HEADER-2x11
- P22: value (none) -> I2S; footprint (none) -> hackrf:GSG-HEADER-2x13
- P25: value (none) -> LPC_ISP; footprint (none) -> hackrf:GSG-HEADER-1x6
- P26: value (none) -> LPC_JTAG; footprint (none) -> hackrf:GSG-50MIL-HEADER-2x5-TH
- P28: value (none) -> SD; footprint (none) -> hackrf:GSG-HEADER-2x11
- P29: value (none) -> CPLD_JTAG; footprint (none) -> hackrf:GSG-HEADER-1x2
- P3: value (none) -> GND; footprint (none) -> hackrf:GSG-HEADER-NOMARK-1x2
- P30: value (none) -> BANK2_AUX; footprint (none) -> hackrf:GSG-HEADER-2x10
- P5: value (none) -> LEDS; footprint (none) -> hackrf:GSG-HEADER-2x3
- P80: value (none) -> SHIELD; footprint (none) -> hackrf:GSG-HEADER-NOMARK-1x2
- Q5: value (none) -> MOSFET_P; footprint (none) -> gsg-modules:SOT23-3
- R100, R19, R30, R34, R77, R78, R79, R80, R81, R86, R87, R88, R89, R90, R91, R96, R98, R99: value (none) -> 39; footprint (none) -> hackrf:GSG-0402
- R12, R37, R48, R49, R51, R52, R54, R59, R62, R63, R64, R66, R67, R68, R7, R93: value (none) -> 10k; footprint (none) -> hackrf:GSG-0402
- R18, R74: value (none) -> 1k8; footprint (none) -> hackrf:GSG-0402
- R46, R55: value (none) -> 162k; footprint (none) -> hackrf:GSG-0402
- R47: value (none) -> 330k; footprint (none) -> hackrf:GSG-0402
- R56: value (none) -> 715k; footprint (none) -> hackrf:GSG-0402
- R57, R58: value (none) -> 0; footprint (none) -> hackrf:GSG-0402
- R65: value (none) -> 18k; footprint (none) -> hackrf:GSG-0402
- R69: value (none) -> 12k; footprint (none) -> hackrf:GSG-0402
- R72, R75: value (none) -> 470; footprint (none) -> hackrf:GSG-0402
- R73, R76: value (none) -> 1k; footprint (none) -> hackrf:GSG-0402
- SW1: value (none) -> DFU; footprint (none) -> hackrf:GSG-SWITCH-FSMRA
- SW2: value (none) -> RESET; footprint (none) -> hackrf:GSG-SWITCH-FSMRA
- U15: value (none) -> TVS; footprint (none) -> hackrf:GSG-LXES1TBCC2-004
- U20: value (none) -> W25Q80; footprint (none) -> hackrf:GSG-SOIC8-208
- U21: value (none) -> TPS62410; footprint (none) -> hackrf:GSG-S-PVSON-N10
- U23: value (none) -> LPC4320FBD144; footprint (none) -> hackrf:GSG-LQFP144
- U24: value (none) -> GSG-XC2C64A-7VQG100C; footprint (none) -> hackrf:GSG-VQ100
- X2: value (none) -> MCU_XTAL; footprint (none) -> hackrf:GSG-XTAL3.2x2.5mm
- X3: value (none) -> RTC_XTAL; footprint (none) -> hackrf:GSG-XTAL-AB26TRQ
